Commit message: Getting arm to work in gazebo

File: catkin/src/cwru_376_student/cwru_urdf/abby_w_arm_urdf.xacro (robot description, xacro)
@@ -785,5 +785,5 @@
   <joint name="kinect_joint" type="fixed">
       <axis xyz="0 1 0" />
-      <origin xyz="0.45 0 1.65" rpy="0 0.92 0"/>
+      <origin xyz="0.45 0 2" rpy="0 0.92 0"/>
       <parent link="base_link"/>
       <child link="kinect_link"/>

Commit message: Fixed xacro merge issue, modified constants for Abby

File: catkin/src/cwru_376_student/cwru_urdf/abby_w_arm_urdf.xacro (robot description, xacro)
@@ -1,1151 +1,167 @@
 <?xml version="1.0" ?>
 <robot
-     xmlns:xacro="http://www.ros.org/wiki/xacro"
-     name="abby">
-   <xacro:property name="track" value=".56515" />
-   <xacro:property name="tirediam" value="0.3302" />
-   <xacro:include filename="$(find abby_description)/urdf/irb120.gazebo" />
-  <!-- Import Rviz colors -->
-  <xacro:include filename="$(find abby_description)/urdf/materials.xacro" />
-   <!--'$(find abby_description)/urdf/irb120.xacro' -->
-   <xacro:include filename="$(find yale_openhand_models)/urdf/wsn_model_t.xacro" />
-  <joint name="gripper_base_joint" type="fixed">
-    <parent link="link7" />
-    <child link="gripper_base_link" />
-    <origin rpy="0 1.5708 0 " xyz="0 0 0"/>
-  </joint>
-	<link name="base_link">
-		<!--visual>
-			<geometry>
-				<mesh filename="package://abby_description/meshes/al_frame_iam_3826baa4.stl" scale="0.0254 0.0254 0.0254"/>
-			</geometry>
-			<origin rpy="0 0 0" xyz="0.0446356739978 0.177065647653 -0.0893087163603"/>
-			<material name="frame1_color">
-				<color rgba="0.752941 0.752941 0.752941 1"/>
-			</material>
-		</visual-->
-		<!--inertial>
-			<mass value="0.01"/>
-			<inertia ixx="0.01" ixy="0.01" ixz="0.01" iyy="0.01" iyz="0.01" izz="0.01"/>
-			<origin rpy="0 0 0" xyz="0 0 0"/>
-		</inertial-->
-	</link>
-		<joint name="base_to_frame1" type="fixed">
-		<parent link="base_link"/>
-		<child link="frame1"/>
-		<!-- z = -0.065 puts x axis right through drive-wheel axle-->
-        <!-- z = 0.105 puts base_link at floor level -->
-        <!-- y = -0.05 to center? 0.26 aligned right side, -0.35 aligned left side, so ctr ~-0.045 -->
-		<origin rpy="0 0 1.5708" xyz="-0.06 -0.045  0.105"/>
-	</joint>
-	<link name="frame1">
-		<visual>
-			<geometry>
-				<mesh filename="package://abby_description/meshes/al_frame_iam_3826baa4.stl" scale="0.0254 0.0254 0.0254"/>
-			</geometry>
-			<origin rpy="0 0 0" xyz="0.0446356739978 0.177065647653 -0.0893087163603"/>
-			<material name="frame1_color">
-				<color rgba="0.752941 0.752941 0.752941 1"/>
-			</material>
-		</visual>
-		<inertial>
-			<mass value="12.7774249075"/>
-			<inertia ixx="2.11995607184" ixy="-0.0128393605839" ixz="-0.0068818565379" iyy="1.84586933127" iyz="0.34872380742" izz="1.11710077832"/>
-			<origin rpy="0 0 0" xyz="0.0382793240557 -0.271251963735 0.649589084908"/>
-		</inertial>
-		<!--collision>
-			<geometry>
-				<mesh filename="package://abby_description/meshes/al_frame_iam_3826baa4.stl" scale="0.0254 0.0254 0.0254"/>
-			</geometry>
-			<origin rpy="0 0 0" xyz="0.0446356739978 0.177065647653 -0.0893087163603"/>
-		</collision-->
-	</link>
-	<link name="f_r_frame_bracket1">
-		<visual>
-			<geometry>
-				<mesh filename="package://abby_description/meshes/frame bracket_ipt_f5a4f28d.stl" scale="0.0254 0.0254 0.0254"/>
-			</geometry>
-			<origin rpy="0 0 0" xyz="-0.0946635865578 -0.0205552039632 -0.424782665556"/>
-			<material name="f_r_frame_bracket1_color">
-				<color rgba="0.639216 0.639216 0.639216 1"/>
-			</material>
-		</visual>
-		<inertial>
-			<mass value="0.71440798275"/>
-			<inertia ixx="0.00043051877529" ixy="0.0" ixz="-1.18150140291e-05" iyy="0.00109167940213" iyz="0.0" izz="0.00105983757016"/>
-			<origin rpy="0 0 0" xyz="-0.0175668955453 0.00484479603152 -0.408054413923"/>
-		</inertial>
-		<!--collision>
-			<geometry>
-				<mesh filename="package://abby_description/meshes/frame bracket_ipt_f5a4f28d.stl" scale="0.0254 0.0254 0.0254"/>
-			</geometry>
-			<origin rpy="0 0 0" xyz="-0.0946635865578 -0.0205552039632 -0.424782665556"/>
-		</collision-->
-	</link>
-	<joint name="frame--f_r_frame_bracket1" type="fixed">
-		<parent link="frame1"/>
-		<child link="f_r_frame_bracket1"/>
-		<origin rpy="0 -0.0938814541614 1.5707963268" xyz="-0.197196963951 -0.46840807491 0.660027160644"/>
-	</joint>
-	<link name="f_l_frame_bracket1">
-		<visual>
-			<geometry>
-				<mesh filename="package://abby_description/meshes/frame bracket_ipt_f5a4f28d.stl" scale="0.0254 0.0254 0.0254"/>
-			</geometry>
-			<origin rpy="0 0 0" xyz="-0.050800692836 -0.0508000000121 -0.00634958439213"/>
-			<material name="f_l_frame_bracket1_color">
-				<color rgba="0.639216 0.639216 0.639216 1"/>
-			</material>
-		</visual>
-		<inertial>
-			<mass value="0.71440798275"/>
-			<inertia ixx="0.00043051877529" ixy="0.0" ixz="-1.18150140291e-05" iyy="0.00109167940213" iyz="0.0" izz="0.00105983757016"/>
-			<origin rpy="0 0 0" xyz="0.026295998169 -0.025399999994 0.0103786672398"/>
-		</inertial>
-		<!--collision>
-			<geometry>
-				<mesh filename="package://abby_description/meshes/frame bracket_ipt_f5a4f28d.stl" scale="0.0254 0.0254 0.0254"/>
-			</geometry>
-			<origin rpy="0 0 0" xyz="-0.050800692836 -0.0508000000121 -0.00634958439213"/>
-		</collision-->
-	</link>
-	<joint name="f_l_frame_bracket--f_r_frame_bracket1" type="fixed">
-		<parent link="f_r_frame_bracket1"/>
-		<child link="f_l_frame_bracket1"/>
-		<origin rpy="0 0 0" xyz="-0.0438628937327 -0.464082383966 -0.418433081198"/>
-	</joint>
-	<link name="f_l_frame_plate1">
-		<visual>
-			<geometry>
-				<mesh filename="package://abby_description/meshes/front frame plate_ipt_3e5bfe16.stl" scale="0.0254 0.0254 0.0254"/>
-			</geometry>
-			<origin rpy="0 0 0" xyz="0 0 0"/>
-			<material name="f_l_frame_plate1_color">
-				<color rgba="0.752941 0.752941 0.752941 1"/>
-			</material>
-		</visual>
-		<inertial>
-			<mass value="0.072583397455"/>
-			<inertia ixx="0.000139975007751" ixy="0.0" ixz="0.0" iyy="3.5475798236e-05" iyz="0.0" izz="0.000174962980108"/>
-			<origin rpy="0 0 0" xyz="0.0380034800186 0.0762017426097 0.00317605933453"/>
-		</inertial>
-		<!--collision>
-			<geometry>
-				<mesh filename="package://abby_description/meshes/front frame plate_ipt_3e5bfe16.stl" scale="0.0254 0.0254 0.0254"/>
-			</geometry>
-			<origin rpy="0 0 0" xyz="0 0 0"/>
-		</collision-->
-	</link>
-	<joint name="f_l_frame_plate--f_l_frame_bracket1" type="fixed">
-		<parent link="f_l_frame_bracket1"/>
-		<child link="f_l_frame_plate1"/>
-		<origin rpy="-3.14159265359 0 1.57079632679" xyz="-0.050800692836 -0.0508000000121 -0.00634958439213"/>
-	</joint>
-	<link name="f_r_frame_plate1">
-		<visual>
-			<geometry>
-				<mesh filename="package://abby_description/meshes/front frame plate_ipt_3e5bfe16.stl" scale="0.0254 0.0254 0.0254"/>
-			</geometry>
-			<origin rpy="0 0 0" xyz="-0.0381000000045 -0.0762009322898 -0.00634941359797"/>
-			<material name="f_r_frame_plate1_color">
-				<color rgba="0.752941 0.752941 0.752941 1"/>
-			</material>
-		</visual>
-		<inertial>
-			<mass value="0.072583397455"/>
-			<inertia ixx="0.000139975007751" ixy="0.0" ixz="0.0" iyy="3.5475798236e-05" iyz="0.0" izz="0.000174962980108"/>
-			<origin rpy="0 0 0" xyz="-9.52500002381e-05 9.97890829302e-07 -0.00317559036918"/>
-		</inertial>
-		<!--collision>
-			<geometry>
-				<mesh filename="package://abby_description/meshes/front frame plate_ipt_3e5bfe16.stl" scale="0.0254 0.0254 0.0254"/>
-			</geometry>
-			<origin rpy="0 0 0" xyz="-0.0381000000045 -0.0762009322898 -0.00634941359797"/>
-		</collision-->
-	</link>
-	<joint name="f_r_frame_plate--f_r_frame_bracket1" type="fixed">
-		<parent link="f_r_frame_bracket1"/>
-		<child link="f_r_frame_plate1"/>
-		<origin rpy="0 0 -1.57079632679" xyz="-0.0184628418291 -0.00785520396718 -0.424783134521"/>
-	</joint>
-	<link name="b_r_frame_bracket1">
-		<visual>
-			<geometry>
-				<mesh filename="package://abby_description/meshes/short frame bracket_ipt_f5a4f28d.stl" scale="0.0254 0.0254 0.0254"/>
-			</geometry>
-			<origin rpy="0 0 0" xyz="-0.0774480173821 -0.0263550400145 -0.00822489041407"/>
-			<material name="b_r_frame_bracket1_color">
-				<color rgba="0.639216 0.639216 0.639216 1"/>
-			</material>
-		</visual>
-		<inertial>
-			<mass value="0.71440798275"/>
-			<inertia ixx="0.00044432538895" ixy="0.0" ixz="-8.3387205787e-05" iyy="0.00086832128551" iyz="0.0" izz="0.00083243813657"/>
-			<origin rpy="0 0 0" xyz="-0.00691246125573 -0.000955040002614 0.00995368760594"/>
-		</inertial>
-		<!--collision>
-			<geometry>
-				<mesh filename="package://abby_description/meshes/short frame bracket_ipt_f5a4f28d.stl" scale="0.0254 0.0254 0.0254"/>
-			</geometry>
-			<origin rpy="0 0 0" xyz="-0.0774480173821 -0.0263550400145 -0.00822489041407"/>
-		</collision-->
-	</link>
-	<joint name="frame--b_r_frame_bracket1" type="fixed">
-		<parent link="frame1"/>
-		<child link="b_r_frame_bracket1"/>
-		<origin rpy="0 -0.0938814541614 1.57079632654" xyz="-0.202996799965 0.113567247403 0.29642350598"/>
-	</joint>
-	<link name="b_r_frame_plate1">
-		<visual>
-			<geometry>
-				<mesh filename="package://abby_description/meshes/back frame plate_ipt_475e4947.stl" scale="0.0254 0.0254 0.0254"/>
-			</geometry>
-			<origin rpy="0 0 0" xyz="-0.0254000000255 -0.126998971214 1.58112569598e-06"/>
-			<material name="b_r_frame_plate1_color">
-				<color rgba="0.752941 0.752941 0.752941 1"/>
-			</material>
-		</visual>
-		<inertial>
-			<mass value="0.0971640215777"/>
-			<inertia ixx="0.0003344255636" ixy="8.4155085275e-07" ixz="0.0" iyy="4.7517225512e-05" iyz="0.0" izz="0.00038129137915"/>
-			<origin rpy="0 0 0" xyz="0.0126431039946 -0.025550836608 0.00317565745359"/>
-		</inertial>
-		<!--collision>
-			<geometry>
-				<mesh filename="package://abby_description/meshes/back frame plate_ipt_475e4947.stl" scale="0.0254 0.0254 0.0254"/>
-			</geometry>
-			<origin rpy="0 0 0" xyz="-0.0254000000255 -0.126998971214 1.58112569598e-06"/>
-		</collision-->
-	</link>
-	<joint name="b_r_frame_plate--b_r_frame_bracket1" type="fixed">
-		<parent link="b_r_frame_bracket1"/>
-		<child link="b_r_frame_plate1"/>
-		<origin rpy="3.14159265359 0 -1.57079632679" xyz="-0.0520471238425 -0.000955040009423 -0.00822349691669"/>
-	</joint>
-	<link name="IRC5_Compact1">
-		<visual>
-			<geometry>
-				<mesh filename="package://abby_description/meshes/irc5_compact_ipt_c844072c.stl" scale="0.0254 0.0254 0.0254"/>
-			</geometry>
-			<origin rpy="0 0 0" xyz="-0.000849884100615 0.0283509919265 -0.462400284136"/>
-			<material name="IRC5_Compact1_color">
-				<color rgba="0.498039 0.498039 0.498039 1"/>
-			</material>
-		</visual>
-		<inertial>
-			<mass value="28.440241599"/>
-			<inertia ixx="0.75499468089" ixy="-0.00122306756239" ixz="-0.00124304296401" iyy="1.08063235538" iyz="-0.0064925615368" izz="0.61093241216"/>
-			<origin rpy="0 0 0" xyz="-0.225686620068 0.151686511222 -0.249482492333"/>
-		</inertial>
-		<!--collision>
-			<geometry>
-				<mesh filename="package://abby_description/meshes/irc5_compact_ipt_c844072c.stl" scale="0.0254 0.0254 0.0254"/>
-			</geometry>
-			<origin rpy="0 0 0" xyz="-0.000849884100615 0.0283509919265 -0.462400284136"/>
-		</collision-->
-	</link>
-	<joint name="frame--IRC5_Compact1" type="fixed">
-		<parent link="frame1"/>
-		<child link="IRC5_Compact1"/>
-		<origin rpy="1.5707959092 0 3.14159265334" xyz="-0.18299683996 0.0935673788127 0.353829950251"/>
-	</joint>
-	<link name="router1">
-		<visual>
-			<geometry>
-				<mesh filename="package://abby_description/meshes/router keepout_ipt_2b3ba7b4.stl" scale="0.0254 0.0254 0.0254"/>
-			</geometry>
-			<origin rpy="0 0 0" xyz="0.0783000719655 0.725341498268 -1.11194969221e-06"/>
-			<material name="router1_color">
-				<color rgba="0.25098 0.321569 0.392157 1"/>
-			</material>
-		</visual>
-		<inertial>
-			<mass value="0.28349523125"/>
-			<inertia ixx="0.00067729370465" ixy="0.0" ixz="0.0" iyy="0.0008954399563" iyz="0.0" izz="0.00150414540089"/>
-			<origin rpy="0 0 0" xyz="0.0783000719663 0.727175853591 0.0190494073449"/>
-		</inertial>
-		<!--collision>
-			<geometry>
-				<mesh filename="package://abby_description/meshes/router keepout_ipt_2b3ba7b4.stl" scale="0.0254 0.0254 0.0254"/>
-			</geometry>
-			<origin rpy="0 0 0" xyz="0.0783000719655 0.725341498268 -1.11194969221e-06"/>
-		</collision-->
-	</link>
-	<joint name="frame--router1" type="fixed">
-		<parent link="frame1"/>
-		<child link="router1"/>
-		<origin rpy="-1.5707959092 0 0" xyz="-0.0354469698523 -0.430316747951 1.61002981286"/>
-	</joint>
-	<link name="SICK_LMS2911">
-		<visual>
-			<geometry>
-				<mesh filename="package://abby_description/meshes/lms291_ipt_2ad4e53c.stl" scale="0.0254 0.0254 0.0254"/>
-			</geometry>
-			<!--origin rpy="1.5708 0 -1.5708" xyz="-0.0683999139953 -0.00245779587475 -0.0929987962566"/-->
-                        <origin rpy="1.5708 0 -1.5708" xyz="-0.06834 -0.00245779587475 0.1"/>
-			<material name="SICK_LMS2911_color">
-				<color rgba="0.752941 0.752941 0.752941 1"/>
-			</material>
-		</visual>
-		<inertial>
-			<mass value="3.71737544502"/>
-			<inertia ixx="0.0174805834039" ixy="-4.4195210288e-07" ixz="4.1599227461e-07" iyy="0.0127643577208" iyz="0.00072853444335" izz="0.0175041992098"/>
-			<origin rpy="0 0 0" xyz="-0.0684016920036 0.0653465146418 -0.0708751847642"/>
-		</inertial>
-		<!--collision>
-			<geometry>
-				<mesh filename="package://abby_description/meshes/sick lms291_ipt_2ad4e53c.stl" scale="0.0254 0.0254 0.0254"/>
-			</geometry>
-			<origin rpy="0 0 0" xyz="-0.0683999139953 -0.00245779587475 -0.0929987962566"/>
-		</collision-->
-	</link>
-	<joint name="frame--SICK_LMS2911" type="fixed">
-            <!-- -->
-      		<axis xyz="0 1 0" />
-      		<origin xyz="0.55 0 0.285" rpy="0 0 0"/>  <!--0.285 seems consistent w/ 14" from lidar bottom to floor on abby-->
-            <!-- -->
-		<!--parent link="frame1"/-->
-                <parent link="base_link"/>
-		<child link="SICK_LMS2911"/>
-		<!--origin rpy="1.5707959092 0 -3.14159265358" xyz="-0.0255468119868 -0.474758386705 0.311455920061"/-->
-	</joint>
- <gazebo reference="SICK_LMS2911">
-    <sensor type="gpu_ray" name="sick_lidar_sensor">
-      <pose>0.13 0 0  0 0 0</pose>
-      <visualize>false</visualize>
-      <update_rate>40</update_rate>
-      <ray>
-        <scan>
-          <horizontal>
-            <samples>181</samples>
-            <resolution>1</resolution>
-            <min_angle>-1.570796</min_angle>
-            <max_angle>1.570796</max_angle>
-          </horizontal>
-        </scan>
-        <range>
-          <min>0.10</min>
-          <max>80.0</max>
-          <resolution>0.01</resolution>
-        </range>
-        <noise>
-          <type>gaussian</type>
-          <!-- Noise parameters based on published spec for Hokuyo laser
-               achieving "+-30mm" accuracy at range < 10m.  A mean of 0.0m and
-               stddev of 0.01m will put 99.7% of samples within 0.03m of the true
-               reading. -->
-          <mean>0.0</mean>
-          <stddev>0.01</stddev>
-        </noise>
-      </ray>
-      <plugin name="gazebo_ros_lidar_controller" filename="libgazebo_ros_gpu_laser.so">
-       <!-- <topicName>/laser/scan</topicName> -->
-                <topicName>/scan</topicName>
-        <frameName>SICK_LMS2911</frameName>
-      </plugin>
-    </sensor>
-  </gazebo>
-	<link name="base_plate1">
-		<visual>
-			<geometry>
-				<mesh filename="package://abby_description/meshes/base plate_iam_348b8023.stl" scale="0.0254 0.0254 0.0254"/>
-			</geometry>
-			<origin rpy="0 0 0" xyz="-0.296284250178 -0.709693779926 -0.581261979343"/>
-			<material name="base_plate1_color">
-				<color rgba="0.752941 0.752941 0.752941 1"/>
-			</material>
-		</visual>
-		<inertial>
-			<mass value="11.253309185"/>
-			<inertia ixx="0.192702049774" ixy="-0.0128927375727" ixz="-0.00057983680454" iyy="0.235790506928" iyz="0.002976996201" izz="0.41200655867"/>
-			<origin rpy="0 0 0" xyz="-0.259429264405 -0.197794168785 -0.0311541484255"/>
-		</inertial>
-		<!--collision>
-			<geometry>
-				<mesh filename="package://abby_description/meshes/base plate_iam_348b8023.stl" scale="0.0254 0.0254 0.0254"/>
-			</geometry>
-			<origin rpy="0 0 0" xyz="-0.296284250178 -0.709693779926 -0.581261979343"/>
-		</collision-->
-	</link>
-	<joint name="frame--base_plate1" type="fixed">
-		<parent link="frame1"/>
-		<child link="base_plate1"/>
-		<origin rpy="0 0 1.5707963268" xyz="-0.182996839959 0.0950674391444 0.365829741316"/>
-	</joint>
-	<link name="top_plate1">
-		<visual>
-			<geometry>
-				<mesh filename="package://abby_description/meshes/top plate_ipt_9041f1eb.stl" scale="0.0254 0.0254 0.0254"/>
-			</geometry>
-			<origin rpy="0 0 0" xyz="-0.039999919998 -0.0370003177082 -0.00635046315153"/>
-			<material name="top_plate1_color">
-				<color rgba="0.2 0.2 0.2 1"/>
-			</material>
-		</visual>
-		<inertial>
-			<mass value="2.41906254029"/>
-			<inertia ixx="0.070476646621" ixy="-3.2774173452e-05" ixz="0.0" iyy="0.05993791034" iyz="0.0" izz="0.130398461926"/>
-			<origin rpy="0 0 0" xyz="0.229580439988 0.257942378411 -0.00317445298106"/>
-		</inertial>
-		<!--collision>
-			<geometry>
-				<mesh filename="package://abby_description/meshes/top plate_ipt_9041f1eb.stl" scale="0.0254 0.0254 0.0254"/>
-			</geometry>
-			<origin rpy="0 0 0" xyz="-0.039999919998 -0.0370003177082 -0.00635046315153"/>
-		</collision-->
-	</link>
-	<joint name="frame--top_plate1" type="fixed">
-		<parent link="frame1"/>
-		<child link="top_plate1"/>
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
Commit message: Path marker not rotating correctly, going too far

File: catkin/src/cwru_376_student/cwru_urdf/abby_w_arm_urdf.xacro (robot description, xacro)
@@ -786,11 +786,7 @@
   <joint name="kinect_joint" type="fixed">
       <axis xyz="0 1 0" />
-<<<<<<< HEAD
-      <origin xyz="0.45 0 2" rpy="0 0.92 0"/>
-=======
       <!--origin xyz="0.55 0.03 1.585" rpy="0.06 0.95 0"/ -->
       <!-- elevate the kinect higher, and slight shift to the right -->
       <origin xyz="0.57 0.02 1.87" rpy="0.04 0.955 0"/>
->>>>>>> 0f2947d8cdda94b7b7f0a907b333fc2fd97deefd
       <parent link="base_link"/>
       <child link="kinect_link"/>
